Commit message: James Anderson: added rosdepts for simulator package

File: Joe_Model/JoeMegaTron.xacro (robot description, xacro)
@@ -82,5 +82,5 @@
 		</gazebo>
 	</xacro:macro>
-<xacro:macro name="BoxBody2" params="name width length height *origin">
+        <xacro:macro name="BoxBody2" params="name width length height *origin">
 		<link name="${name}">
 			<inertial>
